File: BloqueMIC5219.sch (KiCad schematic (older format))
At the start: 3 parts, among them U2 MIC5219-3.3BM5

Commit message: Modificaciones 29 de mayo 2017
Ok
Changed lines of the file:
@@
 LIBS:contrib
 LIBS:valves
-LIBS:open-project
-LIBS:NorBot
 LIBS:ej2cese
 LIBS:FT231XS
@@
 	6100 3550 6200 3550
 $Comp
-L PWR_FLAG #FLG013
-U 1 1 592A84F7
-P 4900 3000
-F 0 "#FLG013" H 4900 3095 50  0001 C CNN
-F 1 "PWR_FLAG" H 4900 3180 50  0000 C CNN
-F 2 "" H 4900 3000 50  0000 C CNN
-F 3 "" H 4900 3000 50  0000 C CNN
-	1    4900 3000
+L PWR_FLAG #FLG014
+U 1 1 592DFCDB
+P 4400 3750
+F 0 "#FLG014" H 4400 3845 50  0001 C CNN
+F 1 "PWR_FLAG" H 4400 3930 50  0000 C CNN
+F 2 "" H 4400 3750 50  0000 C CNN
+F 3 "" H 4400 3750 50  0000 C CNN
+	1    4400 3750
 	1    0    0    -1
 $EndComp
 Wire Wire Line
-	4900 3150 4900 3000
+	4400 3750 4600 3750
+Wire Wire Line
+	4600 3750 4600 3350
+Connection ~ 4600 3350
 $EndSCHEMATC

Commit message: En clase se dio revisión
Se reviso en clase
Parts:
- C1, C2: footprint (none) -> pf:C_0603_HandSoldering
- U2: footprint (none) -> pf:SOIC-8
Changed lines of the file:
@@
 F 0 "U2" H 5400 3750 60  0000 C CNN
 F 1 "MIC5219-3.3BM5" H 5450 2950 60  0000 C CNN
-F 2 "" H 5400 3350 60  0000 C CNN
+F 2 "pf:SOIC-8" H 5400 3350 60  0001 C CNN
 F 3 "" H 5400 3350 60  0000 C CNN
 	1    5400 3350
@@
 $EndComp
 $Comp
-L GND #PWR08
+L GND #PWR011
 U 1 1 5929CF21
 P 4500 3350
-F 0 "#PWR08" H 4500 3100 50  0001 C CNN
+F 0 "#PWR011" H 4500 3100 50  0001 C CNN
 F 1 "GND" H 4500 3200 50  0000 C CNN
 F 2 "" H 4500 3350 50  0000 C CNN
@@
 $EndComp
 $Comp
-L +3.3V #PWR09
+L +3.3V #PWR012
 U 1 1 5929CF65
 P 6250 3050
-F 0 "#PWR09" H 6250 2900 50  0001 C CNN
+F 0 "#PWR012" H 6250 2900 50  0001 C CNN
 F 1 "+3.3V" H 6250 3190 50  0000 C CNN
 F 2 "" H 6250 3050 50  0000 C CNN
@@
 $EndComp
 $Comp
-L +5V #PWR010
+L +5V #PWR013
 U 1 1 5929CF7C
 P 4650 3050
-F 0 "#PWR010" H 4650 2900 50  0001 C CNN
+F 0 "#PWR013" H 4650 2900 50  0001 C CNN
 F 1 "+5V" H 4650 3190 50  0000 C CNN
 F 2 "" H 4650 3050 50  0000 C CNN
@@
 F 0 "C2" H 6425 3450 50  0000 L CNN
 F 1 "C" H 6425 3250 50  0000 L CNN
-F 2 "" H 6438 3200 50  0000 C CNN
+F 2 "pf:C_0603_HandSoldering" H 6438 3200 50  0001 C CNN
 F 3 "" H 6400 3350 50  0000 C CNN
 	1    6400 3350
@@
 F 0 "C1" H 6125 3450 50  0000 L CNN
 F 1 "CP1" H 6125 3250 50  0000 L CNN
-F 2 "" H 6100 3350 50  0000 C CNN
+F 2 "pf:C_0603_HandSoldering" H 6100 3350 50  0001 C CNN
 F 3 "" H 6100 3350 50  0000 C CNN
 	1    6100 3350
@@
 $EndComp
 $Comp
-L GND #PWR011
+L GND #PWR014
 U 1 1 5929D1E4
 P 6100 3550
-F 0 "#PWR011" H 6100 3300 50  0001 C CNN
+F 0 "#PWR014" H 6100 3300 50  0001 C CNN
 F 1 "GND" H 6100 3400 50  0000 C CNN
 F 2 "" H 6100 3550 50  0000 C CNN
@@
 $EndComp
 $Comp
-L GND #PWR012
+L GND #PWR015
 U 1 1 5929D1F8
 P 6400 3550
-F 0 "#PWR012" H 6400 3300 50  0001 C CNN
+F 0 "#PWR015" H 6400 3300 50  0001 C CNN
 F 1 "GND" H 6400 3400 50  0000 C CNN
 F 2 "" H 6400 3550 50  0000 C CNN
@@
 	6100 3550 6200 3550
 $Comp
-L PWR_FLAG #FLG014
+L PWR_FLAG #FLG016
 U 1 1 592DFCDB
 P 4400 3750
-F 0 "#FLG014" H 4400 3845 50  0001 C CNN
+F 0 "#FLG016" H 4400 3845 50  0001 C CNN
 F 1 "PWR_FLAG" H 4400 3930 50  0000 C CNN
 F 2 "" H 4400 3750 50  0000 C CNN
