File: BloqueFT231XS.sch (KiCad schematic (older format))
At the start: 11 parts, among them U3 FT231XS

Commit message: En clase se dio revisión
Se reviso en clase
Parts:
- C3, C4, C5, C6: footprint (none) -> pf:C_0603_HandSoldering
- D1, D2: footprint (none) -> LEDs:LED_1206
- R1, R2: footprint (none) -> pf:R_1206_HandSoldering
- R3, R4: footprint RESC1608X55 -> pf:R_1206_HandSoldering
- U3: footprint SSOP20 -> pf:SP3232ECN-SOIC16N
Connections:
- no-connect marks 5 -> 6
Changed lines of the file:
@@
 F 0 "U3" H 4800 3250 50  0000 L BNN
 F 1 "FT231XS" H 4800 2850 50  0000 L BNN
-F 2 "SSOP20" H 5000 3050 50  0001 L BNN
+F 2 "pf:SP3232ECN-SOIC16N" H 5000 3050 50  0001 L BNN
 F 3 "SSOP-20 FTDI" H 5000 3050 50  0001 L BNN
 F 4 "FT231XS" H 5000 3050 50  0001 L BNN "MP"
@@
 F 0 "C6" H 3675 2400 50  0000 L CNN
 F 1 "0.1uF" H 3675 2200 50  0000 L CNN
-F 2 "" H 3688 2150 50  0000 C CNN
+F 2 "pf:C_0603_HandSoldering" H 3688 2150 50  0001 C CNN
 F 3 "" H 3650 2300 50  0000 C CNN
 	1    3650 2300
@@
 F 0 "R3" H 3650 3009 50  0000 L BNN
 F 1 "27" H 3750 3000 50  0000 L BNN
-F 2 "RESC1608X55" H 3800 2950 50  0001 L BNN
+F 2 "pf:R_1206_HandSoldering" H 3800 2950 50  0001 L BNN
 F 3 "0603 Panasonic" H 3800 2950 50  0001 L BNN
 F 4 "ERJ-3GEYJ270V" H 3800 2950 50  0001 L BNN "MP"
@@
 F 0 "R4" H 3650 3209 50  0000 L BNN
 F 1 "27" H 3750 3200 50  0000 L BNN
-F 2 "RESC1608X55" H 3800 3150 50  0001 L BNN
+F 2 "pf:R_1206_HandSoldering" H 3800 3150 50  0001 L BNN
 F 3 "0603 Panasonic" H 3800 3150 50  0001 L BNN
 F 4 "ERJ-3GEYJ270V" H 3800 3150 50  0001 L BNN "MP"
@@
 F 0 "C4" H 3375 2400 50  0000 L CNN
 F 1 "0.1uF" H 3375 2200 50  0000 L CNN
-F 2 "" H 3388 2150 50  0000 C CNN
+F 2 "pf:C_0603_HandSoldering" H 3388 2150 50  0001 C CNN
 F 3 "" H 3350 2300 50  0000 C CNN
 	1    3350 2300
@@
 F 0 "C3" H 3225 3450 50  0000 L CNN
 F 1 "47pF" H 2900 3350 50  0000 L CNN
-F 2 "" H 3238 3200 50  0000 C CNN
+F 2 "pf:C_0603_HandSoldering" H 3238 3200 50  0001 C CNN
 F 3 "" H 3200 3350 50  0000 C CNN
 	1    3200 3350
@@
 F 0 "C5" H 3475 3450 50  0000 L CNN
 F 1 "47pF" H 3550 3350 50  0000 L CNN
-F 2 "" H 3488 3200 50  0000 C CNN
+F 2 "pf:C_0603_HandSoldering" H 3488 3200 50  0001 C CNN
 F 3 "" H 3450 3350 50  0000 C CNN
 	1    3450 3350
 	1    0    0    -1
 $EndComp
-Text Label 3100 2750 0    60   ~ 0
-GND
-Text Label 3450 3500 0    60   ~ 0
-GND
-Wire Wire Line
-	4100 2350 4050 2350
-Wire Wire Line
-	3650 2150 4100 2150
-Wire Wire Line
-	3950 2150 3950 2750
-Wire Wire Line
-	3950 2550 4100 2550
-Wire Wire Line
-	3950 2750 4100 2750
-Connection ~ 3950 2550
-Connection ~ 3950 2150
-Wire Wire Line
-	3650 2450 3650 2500
-Wire Wire Line
-	4100 2950 4000 2950
-Wire Wire Line
-	4100 3150 4000 3150
-Wire Wire Line
-	3600 2950 3000 2950
-Wire Wire Line
-	3600 3150 3000 3150
-Wire Wire Line
-	3000 2750 3100 2750
-Wire Wire Line
-	3350 2500 3350 2450
-Wire Wire Line
-	3350 2050 3350 2150
-Wire Wire Line
-	3000 2100 3350 2100
-Connection ~ 3350 2100
-Wire Wire Line
-	3200 3200 3200 2950
-Connection ~ 3200 2950
-Wire Wire Line
-	3200 3500 3450 3500
-Wire Wire Line
-	3450 3200 3450 3150
-Connection ~ 3450 3150
 $Comp
 L +3.3V #PWR07
@@
 F 0 "R1" V 3530 4050 50  0000 C CNN
 F 1 "1k" V 3450 4050 50  0000 C CNN
-F 2 "" V 3380 4050 50  0000 C CNN
+F 2 "pf:R_1206_HandSoldering" V 3380 4050 50  0001 C CNN
 F 3 "" H 3450 4050 50  0000 C CNN
 	1    3450 4050
@@
 F 0 "D1" H 3550 3850 50  0000 C CNN
 F 1 "LED" H 3700 3850 50  0000 C CNN
-F 2 "" H 3700 3750 50  0000 C CNN
+F 2 "LEDs:LED_1206" H 3700 3750 50  0001 C CNN
 F 3 "" H 3700 3750 50  0000 C CNN
 	1    3700 3750
@@
 F 0 "D2" H 3900 4050 50  0000 C CNN
 F 1 "LED" H 4050 4050 50  0000 C CNN
-F 2 "" H 3900 3950 50  0000 C CNN
+F 2 "LEDs:LED_1206" H 3900 3950 50  0001 C CNN
 F 3 "" H 3900 3950 50  0000 C CNN
 	1    3900 3950
@@
 F 0 "R2" V 3530 4250 50  0000 C CNN
 F 1 "1k" V 3450 4250 50  0000 C CNN
-F 2 "" V 3380 4250 50  0000 C CNN
+F 2 "pf:R_1206_HandSoldering" V 3380 4250 50  0001 C CNN
 F 3 "" H 3450 4250 50  0000 C CNN
 	1    3450 4250
 	0    1    1    0
 $EndComp
-Wire Wire Line
-	3200 3800 3200 4250
-Wire Wire Line
-	3200 4050 3300 4050
-Wire Wire Line
-	3200 4250 3300 4250
-Connection ~ 3200 4050
-Wire Wire Line
-	3600 4250 3900 4250
-Wire Wire Line
-	3900 4250 3900 4150
-Wire Wire Line
-	3900 3750 4100 3750
-Wire Wire Line
-	3600 4050 3700 4050
-Wire Wire Line
-	3700 4050 3700 3950
-Wire Wire Line
-	3700 3550 4100 3550
 NoConn ~ 4100 3950
 NoConn ~ 4100 3350
-Text Label 5950 3950 0    60   ~ 0
-GND
-Wire Wire Line
-	5900 3950 5950 3950
 NoConn ~ 5900 3550
 NoConn ~ 5900 3350
 NoConn ~ 5900 3150
-Wire Wire Line
-	6150 2150 5900 2150
 Text HLabel 6150 2350 2    60   Input ~ 0
 DOUT
@@
 Text HLabel 6150 2950 2    60   Input ~ 0
 DTS_XBEE
+$Comp
+L GND #PWR08
+U 1 1 5930D968
+P 3400 3550
+F 0 "#PWR08" H 3400 3300 50  0001 C CNN
+F 1 "GND" H 3400 3400 50  0000 C CNN
+F 2 "" H 3400 3550 50  0000 C CNN
+F 3 "" H 3400 3550 50  0000 C CNN
+	1    3400 3550
+	1    0    0    -1
+$EndComp
+Wire Wire Line
+	4100 2350 4050 2350
+Wire Wire Line
+	3650 2150 4100 2150
+Wire Wire Line
+	3950 2150 3950 2750
+Wire Wire Line
+	3950 2550 4100 2550
+Wire Wire Line
+	3950 2750 4100 2750
+Connection ~ 3950 2550
+Connection ~ 3950 2150
+Wire Wire Line
+	3650 2450 3650 2500
+Wire Wire Line
+	4100 2950 4000 2950
+Wire Wire Line
+	4100 3150 4000 3150
+Wire Wire Line
+	3600 2950 3000 2950
+Wire Wire Line
+	3600 3150 3000 3150
+Wire Wire Line
+	3000 2750 3100 2750
+Wire Wire Line
+	3350 2500 3350 2450
+Wire Wire Line
+	3350 2050 3350 2150
+Wire Wire Line
+	3000 2100 3350 2100
+Connection ~ 3350 2100
+Wire Wire Line
+	3200 3200 3200 2950
+Connection ~ 3200 2950
+Wire Wire Line
+	3200 3500 3450 3500
+Wire Wire Line
+	3450 3200 3450 3150
+Connection ~ 3450 3150
+Wire Wire Line
+	3200 3800 3200 4250
+Wire Wire Line
+	3200 4050 3300 4050
+Wire Wire Line
+	3200 4250 3300 4250
+Connection ~ 3200 4050
+Wire Wire Line
+	3600 4250 3900 4250
+Wire Wire Line
+	3900 4250 3900 4150
+Wire Wire Line
+	3900 3750 4100 3750
+Wire Wire Line
+	3600 4050 3700 4050
+Wire Wire Line
+	3700 4050 3700 3950
+Wire Wire Line
+	3700 3550 4100 3550
+Wire Wire Line
+	5900 3950 6100 3950
+Wire Wire Line
+	6150 2150 5900 2150
 Wire Wire Line
 	6150 2350 5900 2350
@@
 Wire Wire Line
 	6150 2950 5900 2950
-Text Label 3100 2500 0    60   ~ 0
-GND
-Wire Wire Line
-	3100 2500 3350 2500
+Wire Wire Line
+	3400 3550 3400 3500
+Connection ~ 3400 3500
+$Comp
+L GND #PWR09
+U 1 1 5930DD2A
+P 6100 4000
+F 0 "#PWR09" H 6100 3750 50  0001 C CNN
+F 1 "GND" H 6100 3850 50  0000 C CNN
+F 2 "" H 6100 4000 50  0000 C CNN
+F 3 "" H 6100 4000 50  0000 C CNN
+	1    6100 4000
+	1    0    0    -1
+$EndComp
+Wire Wire Line
+	6100 3950 6100 4000
+NoConn ~ 5900 3700
 $EndSCHEMATC

Commit message: QuitandoBloques
Se le quitan las hojas de bloques
Other:
- moved on the sheet: C3, C4, C5, C6, D1, D2, R1, R2, R3, R4, U3
