File: BloqueRESET.sch (KiCad schematic (older format))
At the start: 0 parts

Commit message: En clase se dio revisión
Se reviso en clase
Parts:
- added D501, D502: LED, LEDs:LED_1206, symbol LED
- added R501: 330, pf:R_1206_HandSoldering, symbol R
- added R502: 1k, pf:R_1206_HandSoldering, symbol R
- added SW501: SPST, Measurement_Points:Test_Point_2Pads, symbol SPST
Connections:
- new net: D501.2 (A), R501.2
- new net: D502.2 (A), R502.2
- new net +5V: R502.1
- new net GND: D501.1 (K), D502.1 (K), SW501.1
- new net RESET: SW501.2
- new net RSSI_LED_EN: R501.1
Changed lines of the file:
@@
 Comment4 ""
 $EndDescr
+$Comp
+L R R501
+U 1 1 592F637C
+P 4600 4850
+F 0 "R501" V 4680 4850 50  0000 C CNN
+F 1 "330" V 4600 4850 50  0000 C CNN
+F 2 "pf:R_1206_HandSoldering" V 4530 4850 50  0001 C CNN
+F 3 "" H 4600 4850 50  0000 C CNN
+	1    4600 4850
+	1    0    0    -1
+$EndComp
+$Comp
+L R R502
+U 1 1 592F63C0
+P 4950 4850
+F 0 "R502" V 5030 4850 50  0000 C CNN
+F 1 "1k" V 4950 4850 50  0000 C CNN
+F 2 "pf:R_1206_HandSoldering" V 4880 4850 50  0001 C CNN
+F 3 "" H 4950 4850 50  0000 C CNN
+	1    4950 4850
+	1    0    0    -1
+$EndComp
+$Comp
+L LED D501
+U 1 1 592F63ED
+P 4600 5350
+F 0 "D501" H 4600 5450 50  0000 C CNN
+F 1 "LED" H 4600 5250 50  0000 C CNN
+F 2 "LEDs:LED_1206" H 4600 5350 50  0001 C CNN
+F 3 "" H 4600 5350 50  0000 C CNN
+	1    4600 5350
+	0    -1   -1   0
+$EndComp
+$Comp
+L LED D502
+U 1 1 592F646D
+P 4950 5350
+F 0 "D502" H 4950 5450 50  0000 C CNN
+F 1 "LED" H 4950 5250 50  0000 C CNN
+F 2 "LEDs:LED_1206" H 4950 5350 50  0001 C CNN
+F 3 "" H 4950 5350 50  0000 C CNN
+	1    4950 5350
+	0    -1   -1   0
+$EndComp
+$Comp
+L GND #PWR017
+U 1 1 592F64CE
+P 4600 5700
+F 0 "#PWR017" H 4600 5450 50  0001 C CNN
+F 1 "GND" H 4600 5550 50  0000 C CNN
+F 2 "" H 4600 5700 50  0000 C CNN
+F 3 "" H 4600 5700 50  0000 C CNN
+	1    4600 5700
+	1    0    0    -1
+$EndComp
+$Comp
+L GND #PWR018
+U 1 1 592F64F0
+P 4950 5700
+F 0 "#PWR018" H 4950 5450 50  0001 C CNN
+F 1 "GND" H 4950 5550 50  0000 C CNN
+F 2 "" H 4950 5700 50  0000 C CNN
+F 3 "" H 4950 5700 50  0000 C CNN
+	1    4950 5700
+	1    0    0    -1
+$EndComp
+$Comp
+L +5V #PWR019
+U 1 1 592F6559
+P 4950 4550
+F 0 "#PWR019" H 4950 4400 50  0001 C CNN
+F 1 "+5V" H 4950 4690 50  0000 C CNN
+F 2 "" H 4950 4550 50  0000 C CNN
+F 3 "" H 4950 4550 50  0000 C CNN
+	1    4950 4550
+	1    0    0    -1
+$EndComp
+$Comp
+L SPST SW501
+U 1 1 592F6581
+P 5800 5150
+F 0 "SW501" H 5800 5250 50  0000 C CNN
+F 1 "SPST" H 5800 5050 50  0000 C CNN
+F 2 "Measurement_Points:Test_Point_2Pads" H 5800 5150 50  0001 C CNN
+F 3 "" H 5800 5150 50  0000 C CNN
+	1    5800 5150
+	0    -1   -1   0
+$EndComp
+Wire Wire Line
+	4950 5550 4950 5700
+Wire Wire Line
+	4600 5550 4600 5700
+Wire Wire Line
+	4600 5000 4600 5150
+Wire Wire Line
+	4950 5000 4950 5150
+Text HLabel 5650 4400 0    60   Input ~ 0
+RESET
+Wire Wire Line
+	5800 4650 5800 4400
+Wire Wire Line
+	5800 4400 5650 4400
+$Comp
+L GND #PWR020
+U 1 1 592F678C
+P 5800 5750
+F 0 "#PWR020" H 5800 5500 50  0001 C CNN
+F 1 "GND" H 5800 5600 50  0000 C CNN
+F 2 "" H 5800 5750 50  0000 C CNN
+F 3 "" H 5800 5750 50  0000 C CNN
+	1    5800 5750
+	1    0    0    -1
+$EndComp
+Wire Wire Line
+	5800 5750 5800 5650
+Wire Wire Line
+	4950 4700 4950 4550
+Text HLabel 4400 4500 0    60   Input ~ 0
+RSSI_LED_EN
+Wire Wire Line
+	4600 4700 4600 4500
+Wire Wire Line
+	4600 4500 4400 4500
 $EndSCHEMATC
