File: BloqueXBEE-1B3.sch (KiCad schematic (older format))
At the start: 1 part

Commit message: Modificaciones 29 de mayo 2017
Ok
Parts:
- gave numbers to parts that had none: 1
Changed lines of the file:
@@
 LIBS:contrib
 LIBS:valves
-LIBS:open-project
-LIBS:NorBot
 LIBS:ej2cese
 LIBS:FT231XS
@@
 $EndDescr
 $Comp
-L XB24-Z7WIT-004 U?
+L XB24-Z7WIT-004 U4
 U 1 1 592A8847
 P 5900 3600
-F 0 "U?" H 5900 3600 50  0001 L BNN
+F 0 "U4" H 5900 3600 50  0001 L BNN
 F 1 "XB24-Z7WIT-004" H 5900 3600 50  0001 L BNN
 F 2 "DIP-20" H 5900 3600 50  0001 L BNN

Commit message: En clase se dio revisión
Se reviso en clase
Connections:
- net 3.3V renamed +3V3
Changed lines of the file:
@@
 Wire Wire Line
 	6850 4100 6500 4100
+$Comp
+L +3.3V #PWR010
+U 1 1 59316C36
+P 5250 3100
+F 0 "#PWR010" H 5250 2950 50  0001 C CNN
+F 1 "+3.3V" H 5250 3240 50  0000 C CNN
+F 2 "" H 5250 3100 50  0000 C CNN
+F 3 "" H 5250 3100 50  0000 C CNN
+	1    5250 3100
+	1    0    0    -1
+$EndComp
+Wire Wire Line
+	5250 3100 5250 3200
+Connection ~ 5250 3200
 $EndSCHEMATC
