File: ProFinalKicadV1.sch (KiCad schematic (older format))
At the start: 1 part, among them U1 MICRO-B_USB

Commit message: En clase se dio revisión
Se reviso en clase
Parts:
- U1: footprint (none) -> Connect:USB_Micro-B
Connections:
- net BloqueFT231XS/GND renamed GND
- no-connect marks 6 -> 1
Changed lines of the file:
@@
 F0 "BloqueRESET" 60
 F1 "BloqueRESET.sch" 60
+F2 "RESET" I L 5300 4800 60
+F3 "RSSI_LED_EN" I L 5300 5000 60
 $EndSheet
 $Comp
@@
 F 0 "U1" H 1650 2100 50  0000 C CNN
 F 1 "MICRO-B_USB" H 1650 2700 50  0000 C CNN
-F 2 "" H 1650 2400 60  0000 C CNN
+F 2 "Connect:USB_Micro-B" H 1650 2400 60  0001 C CNN
 F 3 "" H 1650 2400 60  0000 C CNN
 	1    1650 2400
@@
 	1    0    0    -1
 $EndComp
-NoConn ~ 4100 2000
-NoConn ~ 4100 2200
-NoConn ~ 4100 2400
-NoConn ~ 4100 2600
-NoConn ~ 4100 2800
 Wire Wire Line
 	2600 2200 1850 2200
@@
 	4100 2200 3950 2200
 Wire Wire Line
-	4100 2400 3950 2400
+	3950 2400 4200 2400
 Wire Wire Line
-	4100 2600 3950 2600
+	3950 2600 4200 2600
 Wire Wire Line
-	4100 2800 3950 2800
+	3950 2800 4650 2800
 Wire Wire Line
-	4100 2000 3950 2000
+	3950 2000 4250 2000
+Text Label 4100 2200 0    60   ~ 0
+DIN
+Text Label 5150 2100 2    60   ~ 0
+DIN
+Wire Wire Line
+	5300 2100 5150 2100
+Text Label 4250 2000 0    60   ~ 0
+DOUT
+Text Label 5150 2000 2    60   ~ 0
+DOUT
+Wire Wire Line
+	5300 2000 5150 2000
+Text Label 2250 4300 0    60   ~ 0
+GND
+Wire Wire Line
+	2550 4300 2250 4300
+Text Label 5000 2800 0    60   ~ 0
+GND
+Wire Wire Line
+	5300 2800 5000 2800
+Text Label 2300 2600 0    60   ~ 0
+GND
+Text Label 2300 4050 0    60   ~ 0
+3.3V
+Wire Wire Line
+	2550 4050 2300 4050
+Text Label 5050 1900 0    60   ~ 0
+3.3V
+Wire Wire Line
+	5300 1900 5050 1900
+Text Label 7000 2300 0    60   ~ 0
+RTS_XBEE
+Text Label 4200 2400 0    60   ~ 0
+RTS_XBEE
+Text Label 4200 2600 0    60   ~ 0
+CTS_XBEE
+Text Label 7000 2700 0    60   ~ 0
+CTS_XBEE
+Wire Wire Line
+	4650 2800 4650 2700
+Wire Wire Line
+	4650 2700 5300 2700
+Wire Wire Line
+	6650 2300 7000 2300
+Wire Wire Line
+	6650 2700 7000 2700
+Text Label 5100 5000 2    60   ~ 0
+RSSI
+Text Label 5150 2400 2    60   ~ 0
+RSSI
+Wire Wire Line
+	5300 2400 5150 2400
+Wire Wire Line
+	5100 5000 5300 5000
+Text Label 5100 4800 2    60   ~ 0
+RESET
+Text Label 5150 2300 2    60   ~ 0
+RESET
+Wire Wire Line
+	5300 2300 5150 2300
+Wire Wire Line
+	5300 4800 5100 4800
 $EndSCHEMATC

Commit message: QuitandoBloques
Se le quitan las hojas de bloques
Parts:
- added C1, C2, C3, C4, C6: C, Capacitors_SMD:C_0603_HandSoldering, symbol C
- added C5: CP1, Capacitors_SMD:CP_Elec_8x10, symbol CP1
- added D1, D2, D3, D4: LED, LEDs:LED_0603_HandSoldering, symbol LED
- added R1, R2, R5, R6: R, Resistors_SMD:R_0603_HandSoldering, symbol R
- added R3, R4: ERJ-3GEYJ270V, RESC1608X55, symbol ERJ-3GEYJ270V
- added SW501: SPST, Measurement_Points:Test_Point_2Pads, symbol SPST
- added U2: MIC5219-3.3BM5, TO_SOT_Packages_SMD:TSOT-23-5_HandSoldering, symbol MIC5219-3.3BM5
- added U3: FT231XS, RF_Modules:Digi_XBee_SMT, symbol FT231XS
- added U4: XB24-Z7WIT-004, Housings_SOIC:SOIC-20W_7.5x12.8mm_Pitch1.27mm, symbol XB24-Z7WIT-004
- added XA1: Conn_Poncho2P_2x_20x2, pf:Conn_Poncho_Derecha, symbol Conn_Poncho2P_2x_20x2
- U1: footprint Connect:USB_Micro-B -> Connect:USB_B
Connections:
- net +5V: now also C1.1, R6.1, U2.1 (VIN), U2.3 (Enable), U3.P12 (VCC), XA1.2 (+5V)
- net CTS_XBEE: now also U3.P6 (CTS#), U4.12
- net DIN: now also U3.P1 (RXD), U4.3, XA1.25 (rs232TXD)
- net DOUT: now also U3.P17 (TXD), U4.2, XA1.23 (rs232RXD)
- net GND: now also C1.2, C2.2, C3.2, C4.2, C5.2, C6.2, D3.1 (K), D4.1 (K), SW501.2, U2.2 (GND), U3.P13 (GND), U4.10, XA1.4 (GND)
- net RESET: now also SW501.1, U4.5
- net RSSI: now also R5.1, U4.6
- net RTS_XBEE: now also U3.P19 (RTS#), U4.16
- net BloqueFT231XS/D+ renamed D+
- net D+: now also C3.1, R4.1
- net BloqueFT231XS/D- renamed D-
- net D-: now also C2.1, R3.1
- new net: XA1.10 (GNDA), XA1.12 (GNDA), XA1.14 (GNDA), XA1.16 (GNDA), XA1.18 (GNDA), XA1.8 (GNDA)
- new net: XA1.20 (GND), XA1.22 (GND), XA1.24 (GND), XA1.26 (GND), XA1.28 (GND), XA1.30 (GND), XA1.32 (GND)
- new net: XA1.38 (GND), XA1.40 (GND)
- new net: C4.1, U3.P10 (3V3OUT), U3.P11 (RESET#), U3.P20 (VCCIO)
- new net: D1.1 (K), U3.P14 (CBUS1)
- new net: D2.1 (K), U3.P7 (CBUS2)
- new net: R4.2, U3.P8 (USBDP)
- new net: R3.2, U3.P9 (USBDM)
- new net: D1.2 (A), R1.1
- new net: D2.2 (A), R2.1
- new net: D3.2 (A), R5.2
- new net: D4.2 (A), R6.2
- new net +3V3: C5.1, C6.1, R1.2, R2.2, U2.5 (OUT), U4.1, XA1.1 (+3.3V)
- new net DIO0: U4.20
- new net DIO1: U4.19
- new net DIO11: U4.7
- new net DIO12: U4.4
- new net DIO2: U4.18
- new net DIO3: U4.17
- new net DIO4: U4.11
- new net DIO5: U4.15
- new net DIO9: U4.13
- new net DTR_XBEE: U3.P18 (DTR#), U4.9
- new net RES1: U4.8
- new net RES2: U4.14
- no-connect marks 1 -> 40
